Commit message: Apply diff drive controller changes from MoveIt config

File: src/stretch_re1_pro_config/description/stretch_base.ros2_control.xacro (robot description, xacro)
@@ -5,8 +5,33 @@
             <hardware>
                 <plugin>fake_components/GenericSystem</plugin>
+                <param name="calculate_dynamics">true</param>
             </hardware>
-            <joint name="position">
-                <!-- <param name="initial_position">0.0 0.0 0.0</param> -->
-                <command_interface name="position" />
+            <!-- Virtual position joint for supporting MoveIt's planar joint type in joint trajectories -->
+            <joint name="position/x">
+                <param name="initial_position">0.0</param>
+                <command_interface name="velocity" />
+                <state_interface name="position"/>
+                <state_interface name="velocity"/>
+            </joint>
+            <joint name="position/y">
+                <param name="initial_position">0.0</param>
+                <command_interface name="velocity" />
+                <state_interface name="position"/>
+                <state_interface name="velocity"/>
+            </joint>
+            <joint name="position/theta">
+                <param name="initial_position">0.0</param>
+                <command_interface name="velocity" />
+                <state_interface name="position"/>
+                <state_interface name="velocity"/>
+            </joint>
+            <!-- Wheel joints used for diff drive controller support -->
+            <joint name="joint_left_wheel">
+                <command_interface name="velocity"/>
+                <state_interface name="position"/>
+                <state_interface name="velocity"/>
+            </joint>
+            <joint name="joint_right_wheel">
+                <command_interface name="velocity"/>
                 <state_interface name="position"/>
                 <state_interface name="velocity"/>
